File: rp2040-kicad-template.kicad_pcb (KiCad board)
At the start: 2 copper layers, 40 x 40 mm, 42 parts, among them U10 PJ-320A, U11 RP2040, U12 XC6206PxxxMR, U13 USB Boot, U14 USBLC6-2SC6, U15 Reset, U16 W25Q16JVUXIQ, U9 TYPE-C-31-M-12, Y2 12MHz - 20pF

Commit message: Use more 0402 footprints for passive components
Parts:
- C21, C22, C25, C27, C39: footprint Capacitor_SMD:C_0603_1608Metric -> Capacitor_SMD:C_0402_1005Metric
- R1, R14, R15, R17, R18: footprint Resistor_SMD:R_0603_1608Metric -> Resistor_SMD:R_0402_1005Metric
- moved C25 71.6 mm to (205.0, 69.5)
- moved C39 67.4 mm to (203.0, 87.5)
- moved C27 2.55 mm to (199.5, 69.5)
