File: rp2040.kicad_sch (KiCad schematic)
At the start: 40 parts, among them U10 PJ-320A, U11 RP2040, U12 XC6206PxxxMR, U13 USB Boot, U14 USBLC6-2SC6, U15 Reset, U16 W25Q16JVUXIQ, U9 TYPE-C-31-M-12, Y2 12MHz - 20pF

Commit message: Update board design rules, use some smaller components, start laying out PCB
Parts:
- R10, R11: footprint Resistor_SMD:R_0603_1608Metric -> Resistor_SMD:R_0402_1005Metric; LCSC C23186 -> C25905
- R12, R13: footprint Resistor_SMD:R_0603_1608Metric -> Resistor_SMD:R_0402_1005Metric; LCSC C25190 -> C25100
Changed lines of the file:
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@@
 			)
 		)
-		(property "Footprint" "Resistor_SMD:R_0603_1608Metric"
+		(property "Footprint" "Resistor_SMD:R_0402_1005Metric"
 			(at 31.75 113.03 0)
 			(effects
@@
 			)
 		)
-		(property "LCSC" "C25190"
+		(property "LCSC" "C25100"
 			(at 31.75 113.03 90)
 			(effects
@@
 			)
 		)
-		(property "Footprint" "Resistor_SMD:R_0603_1608Metric"
+		(property "Footprint" "Resistor_SMD:R_0402_1005Metric"
 			(at 31.75 115.57 0)
 			(effects
@@
 			)
 		)
-		(property "LCSC" "C25190"
+		(property "LCSC" "C25100"
 			(at 31.75 115.57 90)
 			(effects
@@
 			)
 		)
-		(property "Footprint" "Resistor_SMD:R_0603_1608Metric"
+		(property "Footprint" "Resistor_SMD:R_0402_1005Metric"
 			(at 20.32 69.85 0)
 			(effects
@@
 			)
 		)
-		(property "LCSC" "C23186"
+		(property "LCSC" "C25905"
 			(at 20.32 69.85 0)
 			(effects
@@
 			)
 		)
-		(property "Footprint" "Resistor_SMD:R_0603_1608Metric"
+		(property "Footprint" "Resistor_SMD:R_0402_1005Metric"
 			(at 25.4 69.85 0)
 			(effects
@@
 			)
 		)
-		(property "LCSC" "C23186"
+		(property "LCSC" "C25905"
 			(at 25.4 69.85 0)
 			(effects

Commit message: Use more 0402 footprints for passive components
Parts:
- removed C38: 100nF, Capacitor_SMD:C_0402_1005Metric, symbol Device:C_Small
- C21, C22, C39: footprint Capacitor_SMD:C_0603_1608Metric -> Capacitor_SMD:C_0402_1005Metric; LCSC C23630 -> C12530
- C25, C27: footprint Capacitor_SMD:C_0603_1608Metric -> Capacitor_SMD:C_0402_1005Metric; LCSC C1658 -> C1570
- R14, R15: footprint Resistor_SMD:R_0603_1608Metric -> Resistor_SMD:R_0402_1005Metric; LCSC C21190 -> C11702
- R17, R18: footprint Resistor_SMD:R_0603_1608Metric -> Resistor_SMD:R_0402_1005Metric; LCSC C25804 -> C25744
Changed lines of the file:
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@@
 	)
 	(junction
-		(at 274.32 46.99)
-		(diameter 0)
-		(color 0 0 0 0)
-	)
-	(junction
 		(at 218.44 20.32)
 		(diameter 0)
@@
 		(color 0 0 0 0)
 	)
-	(junction
-		(at 270.51 41.91)
-		(diameter 0)
-		(color 0 0 0 0)
-	)
 	(no_connect
 		(at 74.93 62.23)
@@
 		)
 	)
-	(wire
-		(pts
-			(xy 270.51 46.99) (xy 274.32 46.99)
-		)
-		(stroke
-			(width 0)
-			(type default)
-		)
-	)
 	(polyline
 		(pts
@@
 	(wire
 		(pts
-			(xy 266.7 41.91) (xy 270.51 41.91)
+			(xy 266.7 41.91) (xy 274.32 41.91)
 		)
 		(stroke
@@
 		)
 	)
-	(wire
-		(pts
-			(xy 270.51 41.91) (xy 274.32 41.91)
-		)
-		(stroke
-			(width 0)
-			(type default)
-		)
-	)
 	(polyline
 		(pts
@@
 			)
 		)
-		(property "Footprint" "Capacitor_SMD:C_0603_1608Metric"
+		(property "Footprint" "Capacitor_SMD:C_0402_1005Metric"
 			(at 274.32 44.45 0)
 			(effects
@@
 			)
 		)
-		(property "LCSC" "C23630"
+		(property "LCSC" "C12530"
 			(at 274.32 44.45 0)
 			(effects
@@
 			)
 		)
-		(property "Footprint" "Resistor_SMD:R_0603_1608Metric"
+		(property "Footprint" "Resistor_SMD:R_0402_1005Metric"
 			(at 143.51 49.53 0)
 			(effects
@@
 			)
 		)
-		(property "LCSC" "C25804"
+		(property "LCSC" "C25744"
 			(at 143.51 49.53 0)
 			(effects
@@
 	(symbol
 		(lib_id "Device:C_Small")
-		(at 270.51 44.45 0)
-		(unit 1)
-		(exclude_from_sim no)
-		(in_bom yes)
-		(on_board yes)
-		(dnp no)
-		(property "Reference" "C38"
-			(at 261.62 43.18 0)
-			(effects
-				(font
-					(size 1.27 1.27)
-				)
-				(justify left)
-			)
-		)
-		(property "Value" "100nF"
-			(at 261.62 45.72 0)
-			(effects
-				(font
-					(size 1.27 1.27)
-				)
-				(justify left)
-			)
-		)
-		(property "Footprint" "Capacitor_SMD:C_0402_1005Metric"
-			(at 270.51 44.45 0)
-			(effects
-				(font
-					(size 1.27 1.27)
-				)
-				(hide yes)
-			)
-		)
-		(property "Datasheet" "~"
-			(at 270.51 44.45 0)
-			(effects
-				(font
-					(size 1.27 1.27)
-				)
-				(hide yes)
-			)
-		)
-		(property "Description" ""
-			(at 270.51 44.45 0)
-			(effects
-				(font
-					(size 1.27 1.27)
-				)
-				(hide yes)
-			)
-		)
-		(property "LCSC" "C307331"
-			(at 270.51 44.45 0)
-			(effects
-				(font
-					(size 1.27 1.27)
-				)
-				(hide yes)
-			)
-		)
-		(pin "1"
-		)
-		(pin "2"
-		)
-		(instances
-			(project "rp2040-kicad-template"
-				(path "/bab9d4ba-4671-4f57-a245-5e0527b464d7/59d9fd80-c3ab-4343-9591-286205d42abc"
-					(reference "C38")
-					(unit 1)
-				)
-			)
-		)
-	)
-	(symbol
-		(lib_id "Device:C_Small")
 		(at 269.24 22.86 0)
 		(unit 1)
@@
 			)
 		)
-		(property "Footprint" "Resistor_SMD:R_0603_1608Metric"
+		(property "Footprint" "Resistor_SMD:R_0402_1005Metric"
 			(at 33.02 161.29 0)
 			(effects
@@
 			)
 		)
-		(property "LCSC" "C21190"
+		(property "LCSC" "C11702"
 			(at 33.02 161.29 90)
 			(effects
@@
 			)
 		)
-		(property "Footprint" "Capacitor_SMD:C_0603_1608Metric"
+		(property "Footprint" "Capacitor_SMD:C_0402_1005Metric"
 			(at 53.34 90.17 0)
 			(effects
@@
 			)
 		)
-		(property "LCSC" "C23630"
+		(property "LCSC" "C12530"
 			(at 53.34 90.17 0)
 			(effects
@@
 			)
 		)
-		(property "Footprint" "Capacitor_SMD:C_0603_1608Metric"
+		(property "Footprint" "Capacitor_SMD:C_0402_1005Metric"
 			(at 148.59 26.67 0)
 			(effects
@@
 			)
 		)
-		(property "LCSC" "C1658"
+		(property "LCSC" "C1570"
 			(at 148.59 26.67 0)
 			(effects
@@
 			)
 		)
-		(property "Footprint" "Capacitor_SMD:C_0603_1608Metric"
+		(property "Footprint" "Capacitor_SMD:C_0402_1005Metric"
 			(at 45.72 90.17 0)
 			(effects
@@
 			)
 		)
-		(property "LCSC" "C23630"
+		(property "LCSC" "C12530"
 			(at 45.72 90.17 0)
 			(effects
@@
 			)
 		)
-		(property "Footprint" "Resistor_SMD:R_0603_1608Metric"
+		(property "Footprint" "Resistor_SMD:R_0402_1005Metric"
 			(at 106.68 52.07 0)
 			(effects
@@
 			)
 		)
-		(property "LCSC" "C21190"
+		(property "LCSC" "C11702"
 			(at 106.68 52.07 90)
 			(effects
@@
 			)
 		)
-		(property "Footprint" "Resistor_SMD:R_0603_1608Metric"
+		(property "Footprint" "Resistor_SMD:R_0402_1005Metric"
 			(at 205.74 52.07 0)
 			(effects
@@
 			)
 		)
-		(property "LCSC" "C25804"
+		(property "LCSC" "C25744"
 			(at 205.74 52.07 90)
 			(effects
@@
 			)
 		)
-		(property "Footprint" "Capacitor_SMD:C_0603_1608Metric"
+		(property "Footprint" "Capacitor_SMD:C_0402_1005Metric"
 			(at 135.89 26.67 0)
 			(effects
@@
 			)
 		)
-		(property "LCSC" "C1658"
+		(property "LCSC" "C1570"
 			(at 135.89 26.67 0)
 			(effects
